File: EagleProjectsVES/Tranzistory/mericiObvod.brd (EAGLE design)
At the start: 95.2 x 84.8 mm, 107 parts, among them IC1 TLC272D, IC2 TLC272D, IC3 NE555D, IC4 NE555D, IC5 TLC271D, K1 M3XXH, K2 M3XXH, K3 M3XXH, K4 M3XXH, Q1 BD140, T1 BC547, T2 BC547, T3 BC557B, U12V SMKDSP_1,5/2

Commit message: Tranzistory: - opravena dalsi chybka v napojeni emitoru a serioveho rezistoru
Parts:
- moved R33 34.7 mm to (70.2, 17.8), turned to 0 degrees
- moved R36 34.7 mm to (75.2, 52.1), turned to 0 degrees
- moved R43 34.7 mm to (75.2, 17.8), turned to 0 degrees
- moved R7 34.7 mm to (70.2, 52.1), turned to 0 degrees
- moved R16 27.1 mm to (70.2, 48.3), turned to 0 degrees
- moved R31 27.1 mm to (70.2, 21.6), turned to 0 degrees
- moved R35 27.1 mm to (75.2, 48.3), turned to 0 degrees
- moved R40 27.1 mm to (75.2, 21.6), turned to 0 degrees
- moved EMITOR 26.5 mm to (63.5, 52.1)
- moved R17 19.7 mm to (70.2, 44.5), turned to 0 degrees
- moved R32 19.7 mm to (70.2, 25.4), turned to 0 degrees
- moved R34 19.7 mm to (75.2, 44.5), turned to 0 degrees
- moved R41 19.7 mm to (75.2, 25.4), turned to 0 degrees
- moved R18 12.5 mm to (70.2, 40.6), turned to 0 degrees
- moved R29 12.5 mm to (70.2, 29.2), turned to 0 degrees
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Connections:
- removed net N$48: C13.-, C14.2, R3.2, R34.2, R35.2, R36.2, R37.2, R38.2, R39.2, R40.2, R41.2, R42.2, R43.2, UCE1.2, UCE2.2
- new net N$43: EMITOR.MP, IC5.3, R16.1, R17.1, R18.1, R19.1, R29.1, R30.1, R31.1, R32.1, R33.1, R7.1
- net GND: now also C13.-, C14.2, R3.2, R34.2, R35.2, R36.2, R37.2, R38.2, R39.2, R40.2, R41.2, R42.2, R43.2, UCE1.2, UCE2.2; no longer EMITOR.MP, IC5.3, R16.1, R17.1, R18.1, R19.1, R29.1, R30.1, R31.1, R32.1, R33.1, R7.1
Routing:
- net N$48: track 102.7 -> 0.00 mm
- net N$43: track 0.00 -> 60.6 mm
- net GND: track 74.2 -> 93.5 mm, vias 24 -> 15

Commit message: Pridany anglicke prednasky - hotove P1-P3 x rozpracovana P4
Routing:
- net GND: track 93.5 -> 76.3 mm, vias 15 -> 25
Changed lines of the file:
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@@
 <via x="54.61" y="43.815" extent="1-16" drill="0.7"/>
 <wire x1="52.385" y1="43.815" x2="54.61" y2="43.815" width="0.6096" layer="1"/>
-<wire x1="81.28" y1="17.78" x2="76.1975" y2="17.78" width="1.27" layer="1"/>
-<wire x1="76.1975" y1="17.78" x2="76.1975" y2="21.59" width="1.016" layer="1"/>
-<wire x1="76.1975" y1="21.59" x2="76.1975" y2="25.4" width="1.016" layer="1"/>
-<wire x1="76.1975" y1="25.4" x2="76.1975" y2="29.21" width="1.016" layer="1"/>
-<wire x1="76.1975" y1="29.21" x2="76.1975" y2="33.02" width="1.016" layer="1"/>
-<wire x1="76.1975" y1="33.02" x2="76.1975" y2="36.83" width="1.016" layer="1"/>
-<wire x1="76.1975" y1="36.83" x2="76.1975" y2="40.64" width="1.016" layer="1"/>
-<wire x1="76.1975" y1="40.64" x2="76.1975" y2="44.45" width="1.016" layer="1"/>
-<wire x1="76.1975" y1="44.45" x2="76.1975" y2="48.26" width="1.016" layer="1"/>
-<wire x1="76.1975" y1="48.26" x2="76.1975" y2="52.07" width="1.016" layer="1"/>
 <wire x1="45.78" y1="46.355" x2="47.625" y2="46.355" width="0.6096" layer="1"/>
 <wire x1="47.625" y1="46.355" x2="48.26" y2="46.99" width="0.6096" layer="1"/>
+<via x="78.4225" y="52.07" extent="1-16" drill="0.7"/>
+<via x="78.4225" y="48.26" extent="1-16" drill="0.7"/>
+<via x="78.4225" y="44.45" extent="1-16" drill="0.7"/>
+<via x="78.4225" y="40.64" extent="1-16" drill="0.7"/>
+<via x="78.4225" y="36.83" extent="1-16" drill="0.7"/>
+<via x="78.4225" y="33.02" extent="1-16" drill="0.7"/>
+<via x="78.4225" y="29.21" extent="1-16" drill="0.7"/>
+<via x="78.4225" y="25.4" extent="1-16" drill="0.7"/>
+<via x="78.4225" y="21.59" extent="1-16" drill="0.7"/>
+<via x="78.4225" y="17.78" extent="1-16" drill="0.7"/>
+<wire x1="76.1975" y1="52.07" x2="78.4225" y2="52.07" width="0.8128" layer="1"/>
+<wire x1="76.1975" y1="48.26" x2="78.4225" y2="48.26" width="0.8128" layer="1"/>
+<wire x1="76.1975" y1="44.45" x2="78.4225" y2="44.45" width="0.8128" layer="1"/>
+<wire x1="76.1975" y1="40.64" x2="78.4225" y2="40.64" width="0.8128" layer="1"/>
+<wire x1="76.1975" y1="36.83" x2="78.4225" y2="36.83" width="0.8128" layer="1"/>
+<wire x1="76.1975" y1="33.02" x2="78.4225" y2="33.02" width="0.8128" layer="1"/>
+<wire x1="76.1975" y1="29.21" x2="78.4225" y2="29.21" width="0.8128" layer="1"/>
+<wire x1="76.1975" y1="25.4" x2="78.4225" y2="25.4" width="0.8128" layer="1"/>
+<wire x1="76.1975" y1="21.59" x2="78.4225" y2="21.59" width="0.8128" layer="1"/>
+<wire x1="76.1975" y1="17.78" x2="78.4225" y2="17.78" width="0.8128" layer="1"/>
 </signal>
 <signal name="N$10">
